Commit message: [Model][Visualize] use new type of floating-arm

File: urdf/chimera.urdf.xacro (robot description, xacro)
@@ -6,115 +6,15 @@
   <xacro:include filename="$(find dragon)/urdf/dragon_link.urdf.xacro" />
   <!-- spot -->
-  <xacro:include filename="$(find spot_description)/urdf/spot.urdf.xacro" />
-  <!-- attachment -->
-  <link name="grapple_attachment_base_side">
-    <visual>
-      <origin xyz="0.0 0.0 0.0" rpy="0 0 ${-pi/2}" />
-      <geometry>
-        <mesh filename="package://chimera_ros/meshes/grapple_attachment_base_side.dae" />
-      </geometry>
-    </visual>
-  </link>
-  <joint name="grapple_attachment_base_side_joint" type="fixed">
-    <origin xyz="0.1 0.0 0.008" rpy="0 0 ${-pi/2}" />
-    <axis xyz="1 0 0" />
-    <parent link="front_rail" />
-    <child link="grapple_attachment_base_side" />
-  </joint>
-  <link name="grapple_attachment_arm_side">
-    <visual>
-      <origin xyz="0.0 0.0 0.0" rpy="0 ${pi} ${pi/2}" />
-      <geometry>
-        <mesh filename="package://chimera_ros/meshes/grapple_attachment_arm_side.dae" />
-      </geometry>
-    </visual>
-  </link>
+  <xacro:include filename="$(find chimera_ros)/urdf/spot.urdf.xacro" />
+  <!-- free arm -->
+  <xacro:include filename="$(find free_arm_robot)/robots/quad.urdf.xacro" />
   <!-- the following joint should be configurable-->
   <xacro:if value="$(arg fixed_grapple)">
     <joint name="grapple_attachment_joint" type="fixed">
-      <origin xyz="0.0 0.0 -0.004" rpy="0 ${-pi/2} 0" />
+      <origin xyz="0.0 0.0 0.224" rpy="${pi} ${pi/2} 0" />
       <axis xyz="1 0 0" />
-      <parent link="grapple_attachment_base_side" />
-      <child link="grapple_attachment_arm_side" />
+      <parent link="base_fixture" />
+      <child link="link1" />
     </joint>
   </xacro:if>
-  <!-- copy and modify from dragon -->
-  <joint name="joint1_pitch" type="revolute">
-    <limit effort="10.0" lower="${-pi/2}" upper="${pi/2}" velocity="0.1"/>
-    <parent link="grapple_attachment_arm_side"/>
-    <child link="inter_joint1"/>
-    <origin rpy="${pi/2} 0 0" xyz="0.092 0 0"/>
-    <axis xyz="0 1 0"/>
-    <dynamics damping="0.9" friction="0.05"/>
-  </joint>
-  <!-- inter joint -->
-  <link name="inter_joint1">
-    <!-- common inertial -->
-    <inertial>
-      <origin xyz="${inter_joint_x_offset + 3.43 * 0.001} ${-4.27 * 0.001} ${-1.55 * 0.001}" rpy="0 0 0"/>
-      <mass value="0.1329" />
-      <inertia
-          ixx="0.0001" iyy="0.0001" izz="0.0001"
-          ixy="0" ixz="0.0" iyz="0.0"/>
-    </inertial>
-    <visual>
-      <origin rpy="0 0 0" xyz="${inter_joint_x_offset} 0 0"/>
-      <geometry>
-        <mesh filename="package://dragon/urdf/mesh/inter_joint_junction.dae"/>
-      </geometry>
-    </visual>
-  </link>
-  <joint name="joint1_yaw" type="revolute">
-    <limit effort="10.0" lower="${-pi/2}" upper="${pi/2}" velocity="0.1"/>
-    <parent link="inter_joint1"/>
-    <child link="link2"/>
-    <origin rpy="0 0 0" xyz="${2 * inter_joint_x_offset} 0 0"/>
-    <axis xyz="0 0 1"/>
-    <dynamics damping="0.9" friction="0.05"/>
-  </joint>
-  <xacro:dragon_module self="2" child="3" baselink="false" />
-  <xacro:dragon_module self="3" child="3" baselink="false" />
-  <!-- copy from dragon_valve -->
-  <joint name="gripper_joint" type="fixed">
-    <parent link="link3"/>
-    <child link="gripper"/>
-    <origin xyz="0.397 0 0" rpy="0 0 0"/>
-    <axis xyz="0 0 1"/>
-  </joint>
-  <link name="gripper">
-    <visual>
-      <origin xyz="0 0 0" rpy="0 0 0"/>
-      <geometry>
-        <mesh filename="package://dragon_valve/urdf/mesh/valve_gripper.dae"/>
-      </geometry>
-    </visual>
-  </link>
-  <joint name="tip1_joint" type="fixed">
-    <parent link="gripper"/>
-    <child link="tip1"/>
-    <origin xyz="0 0 0.07" rpy="0 0 0"/>
-    <axis xyz="0 0 1"/>
-  </joint>
-  <link name="tip1">
-    <collision>
-      <origin xyz="0.05 0 0" rpy="0 ${pi/2} 0"/>
-      <geometry>
-        <cylinder length="0.1" radius="0.006"/>
-      </geometry>
-    </collision>
-  </link>
-  <joint name="tip2_joint" type="fixed">
-    <parent link="gripper"/>
-    <child link="tip2"/>
-    <origin xyz="0 0 -0.07" rpy="0 0 0"/>
-    <axis xyz="0 0 1"/>
-  </joint>
-  <link name="tip2">
-    <collision>
-      <origin xyz="0.05 0 0" rpy="0 ${pi/2} 0"/>
-      <geometry>
-        <cylinder length="0.1" radius="0.006"/>
-      </geometry>
-    </collision>
-  </link>
 </robot>

File: urdf/spot.urdf.xacro (robot description, xacro)
@@ -5,17 +5,20 @@
   <xacro:include filename="$(find spot_description)/urdf/spot.urdf.xacro" />
   <!-- attachment -->
-  <link name="grapple_attachment_base_side">
+  <link name="base_fixture">
     <visual>
-      <origin xyz="0.0 0.0 0.0" rpy="0 0 ${-pi/2}" />
+      <origin xyz="0.0 0.0 0.0" rpy="0 0 0" />
       <geometry>
-        <mesh filename="package://chimera_ros/meshes/grapple_attachment_base_side.dae" />
+        <mesh filename="package://chimera_ros/meshes/base_fixture.STL" />
       </geometry>
+      <material name="grey">
+        <color rgba="0.3 0.3 0.3 1" />
+      </material>
     </visual>
   </link>
-  <joint name="grapple_attachment_base_side_joint" type="fixed">
-    <origin xyz="0.1 0.0 0.008" rpy="0 0 0" />
+  <joint name="fixture_joint" type="fixed">
+    <origin xyz="-0.1 0.0 0.008" rpy="0 0 0" />
     <axis xyz="1 0 0" />
     <parent link="front_rail" />
-    <child link="grapple_attachment_base_side" />
+    <child link="base_fixture" />
   </joint>
 </robot>
